Commit message: updating xacro

File: aiscbot_descriptioin/aisc.xacro (robot description, xacro)
@@ -1 +1,13 @@
-<?xml version="1.0" ?>
+<?xml version="1.0"?>
+	<robot name="aiscbot">
+		<link name="base_link">
+		</link>
+		<link name="laser">
+		</link>
+		<joint name="base_link_to_laser" type="fixed">
+			<parent link="base_link"/>
+			<child link="laser"/>
+			<origin xyz="0 0 0.12" rpy="0.0 0.0 0.0"/>
+			<axis xyz="0 0 0"/>
+		</joint>
+	</robot>
