Commit message: description , plugins  updated

File: aiscbot_description/urdf/aiscbot.xacro (robot description, xacro)
@@ -35,5 +35,5 @@
       <mesh filename="package://aiscbot_description/meshes/wheel_rf_1.stl" scale="0.001 0.001 0.001"/>
     </geometry>
-    <material name="silver"/>
+    <material name="black"/>
   </visual>
   <collision>
@@ -55,5 +55,5 @@
       <mesh filename="package://aiscbot_description/meshes/wheel_lf_1.stl" scale="0.001 0.001 0.001"/>
     </geometry>
-    <material name="silver"/>
+    <material name="black"/>
   </visual>
   <collision>
@@ -75,5 +75,5 @@
       <mesh filename="package://aiscbot_description/meshes/wheel_rb_1.stl" scale="0.001 0.001 0.001"/>
     </geometry>
-    <material name="silver"/>
+    <material name="black"/>
   </visual>
   <collision>
@@ -95,5 +95,5 @@
       <mesh filename="package://aiscbot_description/meshes/wheel_lb_1.stl" scale="0.001 0.001 0.001"/>
     </geometry>
-    <material name="silver"/>
+    <material name="black"/>
   </visual>
   <collision>
@@ -115,5 +115,5 @@
       <mesh filename="package://aiscbot_description/meshes/lidar_1.stl" scale="0.001 0.001 0.001"/>
     </geometry>
-    <material name="silver"/>
+    <material name="blue"/>
   </visual>
   <collision>
@@ -128,5 +128,5 @@
   <parent link="base_link"/>
   <child link="wheel_rf_1"/>
-  <axis xyz="0.0 -1.0 0.0"/>
+  <axis xyz="0.0 1.0 0.0"/>
 </joint>
 <joint name="Rev2" type="continuous">
@@ -140,5 +140,5 @@
   <parent link="base_link"/>
   <child link="wheel_rb_1"/>
-  <axis xyz="0.0 -1.0 0.0"/>
+  <axis xyz="0.0 1.0 0.0"/>
 </joint>
 <joint name="Rev4" type="continuous">

File: aiscbot_description/urdf/materials.xacro (robot description, xacro)
@@ -4,3 +4,12 @@
   <color rgba="0.700 0.700 0.700 1.000"/>
 </material>
+<material name="black">
+  <color rgba="0.000 0.000 0.000 1.000"/>
+</material>
+<material name="blue">
+  <color rgba="0.000 0.000 1.000 1.000"/>
+</material>
+<material name="red">
+  <color rgba="0.700 0.700 0.700 1.000"/>
+</material>
 </robot>

Commit message: fixed lidar

File: aiscbot_description/urdf/aiscbot.xacro (robot description, xacro)
@@ -2,5 +2,5 @@
 <robot name="aiscbot" xmlns:xacro="http://www.ros.org/wiki/xacro">
 <xacro:include filename="$(find aiscbot_description)/urdf/materials.xacro" />
-<xacro:include filename="$(find aiscbot_description)/urdf/aiscbot.trans" />
+<!--<xacro:include filename="$(find aiscbot_description)/urdf/aiscbot.trans" />-->
 <xacro:include filename="$(find aiscbot_description)/urdf/aiscbot.gazebo" />
 <link name="base_link">
@@ -124,27 +124,27 @@
   </collision>
 </link>
-<joint name="Rev1" type="continuous">
+<joint name="Rev1" type="fixed">
   <origin rpy="0 0 0" xyz="0.06 -0.0515 0.0325"/>
   <parent link="base_link"/>
   <child link="wheel_rf_1"/>
-  <axis xyz="0.0 1.0 0.0"/>
+  <!--<axis xyz="0.0 1.0 0.0"/>-->
 </joint>
-<joint name="Rev2" type="continuous">
+<joint name="Rev2" type="fixed">
   <origin rpy="0 0 0" xyz="0.06 0.0515 0.0325"/>
   <parent link="base_link"/>
   <child link="wheel_lf_1"/>
-  <axis xyz="0.0 1.0 0.0"/>
+  <!--<axis xyz="0.0 1.0 0.0"/>-->
 </joint>
-<joint name="Rev3" type="continuous">
+<joint name="Rev3" type="fixed">
   <origin rpy="0 0 0" xyz="-0.06 -0.0515 0.0325"/>
   <parent link="base_link"/>
   <child link="wheel_rb_1"/>
-  <axis xyz="0.0 1.0 0.0"/>
+  <!--<axis xyz="0.0 1.0 0.0"/>-->
 </joint>
-<joint name="Rev4" type="continuous">
+<joint name="Rev4" type="fixed">
   <origin rpy="0 0 0" xyz="-0.06 0.0515 0.0325"/>
   <parent link="base_link"/>
   <child link="wheel_lb_1"/>
-  <axis xyz="0.0 1.0 0.0"/>
+  <!--<axis xyz="0.0 1.0 0.0"/>-->
 </joint>
 <joint name="Rigid5" type="fixed">

Commit message: updated gazebo and other params

File: aiscbot_description/urdf/aiscbot.xacro (robot description, xacro)
@@ -124,9 +124,14 @@
   </collision>
 </link>
+<joint name="Rigid5" type="fixed">
+  <origin rpy="0 0 0" xyz="0.0 0.0 0.12"/>
+  <parent link="base_link"/>
+  <child link="lidar_1"/>
+</joint>
+<!--
 <joint name="Rev1" type="fixed">
   <origin rpy="0 0 0" xyz="0.06 -0.0515 0.0325"/>
   <parent link="base_link"/>
   <child link="wheel_rf_1"/>
-  <!--<axis xyz="0.0 1.0 0.0"/>-->
 </joint>
 <joint name="Rev2" type="fixed">
@@ -134,5 +139,4 @@
   <parent link="base_link"/>
   <child link="wheel_lf_1"/>
-  <!--<axis xyz="0.0 1.0 0.0"/>-->
 </joint>
 <joint name="Rev3" type="fixed">
@@ -140,5 +144,4 @@
   <parent link="base_link"/>
   <child link="wheel_rb_1"/>
-  <!--<axis xyz="0.0 1.0 0.0"/>-->
 </joint>
 <joint name="Rev4" type="fixed">
@@ -146,10 +149,29 @@
   <parent link="base_link"/>
   <child link="wheel_lb_1"/>
-  <!--<axis xyz="0.0 1.0 0.0"/>-->
 </joint>
-<joint name="Rigid5" type="fixed">
-  <origin rpy="0 0 0" xyz="0.0 0.0 0.12"/>
+-->
+<joint name="Rev1" type="continuous">
+  <origin rpy="0 0 0" xyz="0.06 -0.0515 0.0325"/>
   <parent link="base_link"/>
-  <child link="lidar_1"/>
+  <child link="wheel_rf_1"/>
+  <axis xyz="0.0 1.0 0.0"/>
+</joint>
+<joint name="Rev2" type="continuous">
+  <origin rpy="0 0 0" xyz="0.06 0.0515 0.0325"/>
+  <parent link="base_link"/>
+  <child link="wheel_lf_1"/>
+  <axis xyz="0.0 1.0 0.0"/>
+</joint>
+<joint name="Rev3" type="continuous">
+  <origin rpy="0 0 0" xyz="-0.06 -0.0515 0.0325"/>
+  <parent link="base_link"/>
+  <child link="wheel_rb_1"/>
+  <axis xyz="0.0 1.0 0.0"/>
+</joint>
+<joint name="Rev4" type="continuous">
+  <origin rpy="0 0 0" xyz="-0.06 0.0515 0.0325"/>
+  <parent link="base_link"/>
+  <child link="wheel_lb_1"/>
+  <axis xyz="0.0 1.0 0.0"/>
 </joint>
 </robot>
